File: KiCad/Econet clock 2_2.kicad_sch (KiCad schematic)
At the start: 17 parts, among them IC1 ATtiny45-20PU, J1 Conn_01x02_Male, J2 Conn_01x02_Pin, J3 Conn_01x06_Pin, SW1 SW_DIP_x04

Commit message: Updated data polarity markings, increased decoupling capacitance
Parts:
- C1: value 10uF -> 22uF
- SV1: value Ext DIN header 1 -> Header 1
- SV2: value Ext DIN Header 2 -> Header 2
Connections:
- net CLK+: now also SV1.2 (Pin_2), SV2.2 (Pin_2); no longer SV1.4 (Pin_4), SV2.4 (Pin_4)
- net CLK-: now also SV1.1 (Pin_1), SV2.1 (Pin_1); no longer SV1.5 (Pin_5), SV2.5 (Pin_5)
- net DATA+: now also SV1.4 (Pin_4), SV2.4 (Pin_4), SV3.1, SV4.1; no longer SV1.1 (Pin_1), SV2.1 (Pin_1), SV3.4, SV4.4
- net DATA-: now also SV1.5 (Pin_5), SV2.5 (Pin_5), SV3.4, SV4.4; no longer SV1.2 (Pin_2), SV2.2 (Pin_2), SV3.1, SV4.1
Other:
- moved on the sheet: SV1, SV2
Changed lines of the file:
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@@
 	)
 	(label "DATA+"
-		(at 207.01 88.9 0)
+		(at 215.9 86.36 0)
 		(effects
 			(font
@@
 	)
 	(label "DATA-"
-		(at 215.9 86.36 0)
+		(at 207.01 88.9 0)
 		(effects
 			(font
@@
 			)
 		)
-		(property "Value" "10uF"
+		(property "Value" "22uF"
 			(at 75.184 119.38 0)
 			(effects
@@
 	(symbol
 		(lib_id "Connector:Conn_01x05_Pin")
-		(at 200.66 33.02 180)
+		(at 200.66 33.02 0)
+		(mirror y)
 		(unit 1)
 		(exclude_from_sim no)
@@
 			)
 		)
-		(property "Value" "Ext DIN header 1"
-			(at 201.93 22.86 0)
+		(property "Value" "Header 1"
+			(at 195.072 26.67 0)
 			(effects
 				(font
@@
 	(symbol
 		(lib_id "Connector:Conn_01x05_Pin")
-		(at 200.66 55.88 180)
+		(at 200.66 55.88 0)
+		(mirror y)
 		(unit 1)
 		(exclude_from_sim no)
@@
 			)
 		)
-		(property "Value" "Ext DIN Header 2"
-			(at 201.93 45.72 0)
-			(effects
-				(font
+		(property "Value" "Header 2"
+			(at 195.072 49.53 0)
+			(effects
+				(font
